Commit message: fixed controllers for joints

File: urdf/main.xacro (robot description, xacro)
@@ -2,5 +2,5 @@
 <robot xmlns:xacro="http://www.ros.org/wiki/xacro" name="my_robot">
     <xacro:include filename="$(find project_rp)/urdf/r_link.xacro" />
-    <link name="base_link">
+    <link name="base">
         <visual>
             <geometry>
@@ -18,7 +18,7 @@
         </inertial>
     </link>
-    <xacro:r_link prefix="l1" parent="base_link" length="1.0" radius=".1" rpy="0 0 0" joint_xyz="0 0 0.05" link_xyz="0 0 0.5"/>
-    <xacro:r_link prefix="l2" parent="l1_link" length=".3" radius=".1" rpy="0 ${pi/2} 0" joint_xyz="0 0 1" link_xyz="0 0 0" />
-    <xacro:r_link prefix="l3" parent="l2_link" length="1.0" radius=".075" rpy="0 ${-pi/2} 0" joint_xyz="0 0 0" link_xyz="0 0 0.5" />
+    <xacro:r_link prefix="l1" parent="base" length="1.0" radius=".1" rpy="0 0 0" joint_xyz="0 0 0.05" link_xyz="0 0 0.5"/>
+    <xacro:r_link prefix="l2" parent="l1" length=".3" radius=".1" rpy="0 ${pi/2} 0" joint_xyz="0 0 1" link_xyz="0 0 0" />
+    <xacro:r_link prefix="l3" parent="l2" length="1.0" radius=".075" rpy="0 ${-pi/2} 0" joint_xyz="0 0 0" link_xyz="0 0 0.5" />
     <!-- Add ROS plugin so we can interact with our robot -->
     <gazebo>

File: urdf/r_link.xacro (robot description, xacro)
@@ -4,5 +4,5 @@
     <!-- rpy (roll pitch yaw) describes rotation in radians -->
     <!-- xyz describes translation in meters -->
-    <link name="${prefix}_link">
+    <link name="${prefix}">
         <visual>
             <origin rpy="0 0 0" xyz="${link_xyz}"/> <!-- set the origin to 0 to recenter the link to the child_frame -->
@@ -23,8 +23,8 @@
         </inertial>
     </link>
-    <joint name="base_to_${prefix}" type="revolute">
+    <joint name="${parent}_to_${prefix}" type="continuous">
         <axis xyz="0 0 1"/>
         <parent link="${parent}"/>
-        <child link="${prefix}_link"/>
+        <child link="${prefix}"/>
         <origin rpy="${rpy}" xyz="${joint_xyz}"/> <!-- move the child_frame with respect to parent_frame -->
         <limit effort="30" velocity="1.0"/>
@@ -35,5 +35,5 @@
             <mechanicalReduction>1</mechanicalReduction>
         </actuator>
-        <joint name="base_to_${prefix}">
+        <joint name="${parent}_to_${prefix}">
             <hardwareInterface>hardware_interface/PositionJointInterface</hardwareInterface>
         </joint>

Commit message: make manipulator now generates main.xacro file from input DH_params.txt file. Also made changes on r_link.xacro and base.xacro.

File: urdf/main.xacro (robot description, xacro)
@@ -2,24 +2,11 @@
 <robot xmlns:xacro="http://www.ros.org/wiki/xacro" name="my_robot">
     <xacro:include filename="$(find project_rp)/urdf/r_link.xacro" />
-    <link name="base">
-        <visual>
-            <geometry>
-                <box size="1 1 .1"/>
-            </geometry>
-        </visual>
-        <collision>
-            <geometry>
-                <box size="1 1 .1"/>
-            </geometry>
-        </collision>
-        <inertial>
-            <mass value="1"/>
-            <inertia ixx="0.21" ixy="0" ixz="0" iyy="0.27" iyz="0" izz="0.10"/>
-        </inertial>
-    </link>
-    <xacro:r_link prefix="l1" parent="base" length="1.0" radius=".1" rpy="0 0 0" joint_xyz="0 0 0.05" link_xyz="0 0 0.5"/>
-    <xacro:r_link prefix="l2" parent="l1" length=".3" radius=".1" rpy="0 ${pi/2} 0" joint_xyz="0 0 1" link_xyz="0 0 0" />
-    <xacro:r_link prefix="l3" parent="l2" length="1.0" radius=".075" rpy="0 ${-pi/2} 0" joint_xyz="0 0 0" link_xyz="0 0 0.5" />
-    <!-- Add ROS plugin so we can interact with our robot -->
+    <xacro:include filename="$(find project_rp)/urdf/base.xacro" />
+    <xacro:base name="l0" />
+    <xacro:r_link prefix="l1" parent="l0" length="1.400000" radius="0.1" joint_rpy="0 0 0" joint_xyz="0 0 0" link_rpy="0 0 0" link_xyz="0 0 0.700000" type="revolute"/>
+    <xacro:r_link prefix="l2" parent="l1" length="0.2" radius="0.1" joint_rpy="-1.570796 0 0" joint_xyz="0 0 1.400000" link_rpy="0 0 0" link_xyz="0 0 0.000000" type="revolute"/>
+    <xacro:r_link prefix="l3" parent="l2" length="1.200000" radius="0.1" joint_rpy="1.570796 0 0" joint_xyz="0 0 0.000000" link_rpy="0 0 0" link_xyz="0 0 0.600000" type="revolute"/>
+    <xacro:r_link prefix="l4" parent="l3" length="0.2" radius="0.1" joint_rpy="-1.570796 0 0" joint_xyz="0 0 1.200000" link_rpy="0 0 0" link_xyz="0 0 0.000000" type="revolute"/>
+    <xacro:r_link prefix="l5" parent="l4" length="1.000000" radius="0.1" joint_rpy="0.000000 0 0" joint_xyz="0 0 0" link_rpy="0 1.570796 0" link_xyz="0.500000 0 0" type="revolute"/>
     <gazebo>
         <plugin name="gazebo_ros_control" filename="libgazebo_ros_control.so">

File: urdf/r_link.xacro (robot description, xacro)
@@ -1,10 +1,8 @@
 <?xml version="1.0"?>
 <robot xmlns:xacro="http://www.ros.org/wiki/xacro" name="my_robot">
-<xacro:macro name="r_link" params="prefix parent length radius rpy joint_xyz link_xyz">
-    <!-- rpy (roll pitch yaw) describes rotation in radians -->
-    <!-- xyz describes translation in meters -->
+<xacro:macro name="r_link" params="prefix parent length radius joint_rpy joint_xyz link_rpy link_xyz type">
     <link name="${prefix}">
         <visual>
-            <origin rpy="0 0 0" xyz="${link_xyz}"/> <!-- set the origin to 0 to recenter the link to the child_frame -->
+            <origin rpy="${link_rpy}" xyz="${link_xyz}"/> <!-- set the origin to 0 to recenter the link to the child_frame -->
             <geometry>
                 <cylinder length="${length}" radius="${radius}"/>
@@ -12,5 +10,5 @@
         </visual>
         <collision>
-            <origin rpy="0 0 0" xyz="${link_xyz}"/> <!-- set the origin to 0 to recenter the link to the child_frame -->
+            <origin rpy="${link_rpy}" xyz="${link_xyz}"/> <!-- set the origin to 0 to recenter the link to the child_frame -->
             <geometry>
                 <cylinder length="${length}" radius="${radius}"/>
@@ -18,14 +16,14 @@
         </collision>
         <inertial>
-            <origin rpy="0 0 0" xyz="${link_xyz}"/> <!-- set the origin to 0 to recenter the link to the child_frame -->
+            <origin rpy="${link_rpy}" xyz="${link_xyz}"/> <!-- set the origin to 0 to recenter the link to the child_frame -->
             <mass value="1"/>
             <inertia ixx="0.06" ixy="0.0" ixz="0.0" iyy="0.06" iyz="0.0" izz="0.25"/>
         </inertial>
     </link>
-    <joint name="${parent}_to_${prefix}" type="continuous">
+    <joint name="${parent}_to_${prefix}" type="${type}">
         <axis xyz="0 0 1"/>
         <parent link="${parent}"/>
         <child link="${prefix}"/>
-        <origin rpy="${rpy}" xyz="${joint_xyz}"/> <!-- move the child_frame with respect to parent_frame -->
+        <origin rpy="${joint_rpy}" xyz="${joint_xyz}"/> <!-- move the child_frame with respect to parent_frame -->
         <limit effort="30" velocity="1.0"/>
     </joint>
