Commit message: fixed robot base to the world. Changed spawning position

File: urdf/base.xacro (robot description, xacro)
@@ -2,17 +2,23 @@
 <robot xmlns:xacro="http://www.ros.org/wiki/xacro" name="my_robot">
 <xacro:macro name="base" params="name">
+		<link name="world"/>
+		<joint name="fixed" type="fixed">
+			<parent link="world"/>
+			<child link="${name}"/>
+		</joint>
 		<link name="${name}">
         <visual>
+        		<origin xyz="0 0 0"/>
             <geometry>
-                <box size="2 2 .1"/>
+                <box size="2 2 0"/>
             </geometry>
         </visual>
         <collision>
             <geometry>
-                <box size="2 2 .1"/>
+                <box size="2 2 0"/>
             </geometry>
         </collision>
         <inertial>
-            <mass value="5"/>
+            <mass value="1"/>
             <inertia ixx="0.21" ixy="0" ixz="0" iyy="0.27" iyz="0" izz="0.10"/>
         </inertial>
