Commit message: added prismatic joint macro. added prismatic joint support in make_manipulator. added fixed links for shoulders. broken set_joints!

File: urdf/f_link.xacro (robot description, xacro)
@@ -9,10 +9,4 @@
             </geometry>
         </visual>
-        <collision>
-            <origin rpy="${link_rpy}" xyz="${link_xyz}"/>
-            <geometry>
-                <cylinder length="${length}" radius="${radius}"/>
-            </geometry>
-        </collision>
         <inertial>
             <origin rpy="${link_rpy}" xyz="${link_xyz}"/>

File: urdf/main.xacro (robot description, xacro)
@@ -2,12 +2,15 @@
 <robot xmlns:xacro="http://www.ros.org/wiki/xacro" name="my_robot">
     <xacro:include filename="$(find project_rp)/urdf/r_link.xacro" />
+    <xacro:include filename="$(find project_rp)/urdf/p_link.xacro" />
     <xacro:include filename="$(find project_rp)/urdf/f_link.xacro" />
     <xacro:include filename="$(find project_rp)/urdf/base.xacro" />
     <xacro:base name="l0" />
-    <xacro:r_link prefix="l1" parent="l0" length="1.400000" radius="0.1" joint_rpy="0 0 0" joint_xyz="0 0 0" link_rpy="0 0 0" link_xyz="0 0 0.700000" type="continuous"/>
-    <xacro:r_link prefix="l2" parent="l1" length="0.2" radius="0.1" joint_rpy="-1.570796 0 0" joint_xyz="0.000000 0 1.400000" link_rpy="0 0 0" link_xyz="0.000000 0 0.000000" type="continuous"/>
-    <xacro:r_link prefix="l3" parent="l2" length="1.200000" radius="0.1" joint_rpy="1.570796 0 0" joint_xyz="0.000000 0 0.000000" link_rpy="0 0 0" link_xyz="0.000000 0 0.600000" type="continuous"/>
-    <xacro:r_link prefix="l4" parent="l3" length="0.2" radius="0.1" joint_rpy="-1.570796 0 0" joint_xyz="0.000000 0 1.200000" link_rpy="0 0 0" link_xyz="0.000000 0 0.000000" type="continuous"/>
-    <xacro:f_link prefix="l5" parent="l4" length="1.000000" radius="0.1" link_rpy="0 1.570796 0" link_xyz="0.500000 0 0.000000"/>
+    <xacro:r_link prefix="l1" parent="l0" length="1.000000" radius="0.1" joint_rpy="0 0 0" joint_xyz="0 0 0" link_rpy="0 0 0" link_xyz="0 0 0.500000"/>
+    <xacro:f_link prefix="l2" parent="l1" length="0.200000" radius="0.1" link_rpy="0 1.570796 0" link_xyz="0.100000 0 1.000000"/>
+    <xacro:r_link prefix="l3" parent="l2" length="0.2" radius="0.1" joint_rpy="1.570796 0 0" joint_xyz="0.200000 0 1.000000" link_rpy="0 0 0" link_xyz="0 0 0.000000"/>
+    <xacro:f_link prefix="l4" parent="l3" length="1.000000" radius="0.1" link_rpy="0 1.570796 0" link_xyz="0.500000 0 0.000000"/>
+    <xacro:r_link prefix="l5" parent="l4" length="0.2" radius="0.1" joint_rpy="0.000000 0 0" joint_xyz="1.000000 0 0.000000" link_rpy="0 0 0" link_xyz="0 0 0.000000"/>
+    <xacro:f_link prefix="l6" parent="l5" length="0.200000" radius="0.1" link_rpy="0 1.570796 0" link_xyz="0.100000 0 0.000000"/>
+    <xacro:p_link prefix="l7" parent="l6" length="1.0" radius="0.08" joint_rpy="1.570796 0 0" joint_xyz="0.200000 0 0.000000" link_rpy="0 0 0" link_xyz="0 0 -0.500000"/>
     <gazebo>
         <plugin name="gazebo_ros_control" filename="libgazebo_ros_control.so">

File: urdf/p_link.xacro (robot description, xacro)
@@ -1,5 +1,5 @@
 <?xml version="1.0"?>
 <robot xmlns:xacro="http://www.ros.org/wiki/xacro" name="my_robot">
-<xacro:macro name="r_link" params="prefix parent length radius joint_rpy joint_xyz link_rpy link_xyz">
+<xacro:macro name="p_link" params="prefix parent length radius joint_rpy joint_xyz link_rpy link_xyz">
     <link name="${prefix}">
         <visual>
@@ -15,10 +15,10 @@
         </inertial>
     </link>
-    <joint name="${parent}_to_${prefix}" type="continuous">
+    <joint name="${parent}_to_${prefix}" type="prismatic">
         <axis xyz="0 0 1"/>
         <parent link="${parent}"/>
         <child link="${prefix}"/>
-        <origin rpy="${joint_rpy}" xyz="${joint_xyz}"/>
-        <limit effort="30" velocity="1.0"/>
+        <origin rpy="${joint_rpy}" xyz="${joint_xyz}"/> <!-- move the child_frame with respect to parent_frame -->
+        <limit upper="1" effort="30" velocity="1.0"/>
     </joint>
     <transmission name="${prefix}_transmission">

Commit message: added dampening to improve joint stability

File: urdf/f_link.xacro (robot description, xacro)
@@ -18,4 +18,5 @@
 			<parent link="${parent}"/>
 			<child link="${prefix}"/>
+			<dynamics damping="0.5" friction="0.0"/>
 		</joint>
 </xacro:macro>

File: urdf/main.xacro (robot description, xacro)
@@ -6,11 +6,11 @@
     <xacro:include filename="$(find project_rp)/urdf/base.xacro" />
     <xacro:base name="l0" />
-    <xacro:r_link prefix="l1" parent="l0" length="1.000000" radius="0.1" joint_rpy="0 0 0" joint_xyz="0 0 0" link_rpy="0 0 0" link_xyz="0 0 0.500000"/>
-    <xacro:f_link prefix="l2" parent="l1" length="0.200000" radius="0.1" link_rpy="0 1.570796 0" link_xyz="0.100000 0 1.000000"/>
-    <xacro:r_link prefix="l3" parent="l2" length="0.2" radius="0.1" joint_rpy="1.570796 0 0" joint_xyz="0.200000 0 1.000000" link_rpy="0 0 0" link_xyz="0 0 0.000000"/>
-    <xacro:f_link prefix="l4" parent="l3" length="1.000000" radius="0.1" link_rpy="0 1.570796 0" link_xyz="0.500000 0 0.000000"/>
-    <xacro:r_link prefix="l5" parent="l4" length="0.2" radius="0.1" joint_rpy="0.000000 0 0" joint_xyz="1.000000 0 0.000000" link_rpy="0 0 0" link_xyz="0 0 0.000000"/>
-    <xacro:f_link prefix="l6" parent="l5" length="0.200000" radius="0.1" link_rpy="0 1.570796 0" link_xyz="0.100000 0 0.000000"/>
-    <xacro:p_link prefix="l7" parent="l6" length="1.0" radius="0.08" joint_rpy="1.570796 0 0" joint_xyz="0.200000 0 0.000000" link_rpy="0 0 0" link_xyz="0 0 -0.500000"/>
+    <xacro:r_link prefix="l1" parent="l0" length="1.000000" radius="0.100000" joint_rpy="0 0 0" joint_xyz="0 0 0" link_rpy="0 0 0" link_xyz="0 0 0.500000"/>
+    <xacro:f_link prefix="l2" parent="l1" length="0.200000" radius="0.100000" link_rpy="0 1.570796 0" link_xyz="0.100000 0 1.000000"/>
+    <xacro:r_link prefix="l3" parent="l2" length="0.2" radius="0.100000" joint_rpy="1.570796 0 0" joint_xyz="0.200000 0 1.000000" link_rpy="0 0 0" link_xyz="0 0 0.000000"/>
+    <xacro:f_link prefix="l4" parent="l3" length="1.000000" radius="0.100000" link_rpy="0 1.570796 0" link_xyz="0.500000 0 0.000000"/>
+    <xacro:r_link prefix="l5" parent="l4" length="0.2" radius="0.100000" joint_rpy="0.000000 0 0" joint_xyz="1.000000 0 0.000000" link_rpy="0 0 0" link_xyz="0 0 0.000000"/>
+    <xacro:f_link prefix="l6" parent="l5" length="0.200000" radius="0.100000" link_rpy="0 1.570796 0" link_xyz="0.100000 0 0.000000"/>
+    <xacro:p_link prefix="l7" parent="l6" length="1.500000" radius="0.080000" joint_rpy="1.570796 0 0" joint_xyz="0.200000 0 0.000000" link_rpy="0 0 0" link_xyz="0 0 -0.750000"/>
     <gazebo>
         <plugin name="gazebo_ros_control" filename="libgazebo_ros_control.so">

File: urdf/p_link.xacro (robot description, xacro)
@@ -20,5 +20,6 @@
         <child link="${prefix}"/>
         <origin rpy="${joint_rpy}" xyz="${joint_xyz}"/> <!-- move the child_frame with respect to parent_frame -->
-        <limit upper="1" effort="30" velocity="1.0"/>
+        <limit upper="${length}" effort="30" velocity="1.0"/>
+        <dynamics damping="0.5" friction="0.0"/>
     </joint>
     <transmission name="${prefix}_transmission">

File: urdf/r_link.xacro (robot description, xacro)
@@ -21,4 +21,5 @@
         <origin rpy="${joint_rpy}" xyz="${joint_xyz}"/>
         <limit effort="30" velocity="1.0"/>
+        <dynamics damping="0.5" friction="0.0"/>
     </joint>
     <transmission name="${prefix}_transmission">

Commit message: added claw to the end effector. changed makemanipulator to account for that

File: urdf/f_link.xacro (robot description, xacro)
@@ -1,5 +1,5 @@
 <?xml version="1.0"?>
 <robot xmlns:xacro="http://www.ros.org/wiki/xacro" name="my_robot">
-<xacro:macro name="f_link" params="prefix parent length radius link_rpy link_xyz">
+<xacro:macro name="f_link" params="prefix parent length radius joint_xyz link_rpy link_xyz">
 		<link name="${prefix}">
         <visual>
@@ -18,4 +18,5 @@
 			<parent link="${parent}"/>
 			<child link="${prefix}"/>
+			<origin rpy="0 0 0" xyz="${joint_xyz}"/>
 			<dynamics damping="0.5" friction="0.0"/>
 		</joint>

File: urdf/main.xacro (robot description, xacro)
@@ -5,12 +5,16 @@
     <xacro:include filename="$(find project_rp)/urdf/f_link.xacro" />
     <xacro:include filename="$(find project_rp)/urdf/base.xacro" />
+    <xacro:include filename="$(find project_rp)/urdf/claw.xacro" />
     <xacro:base name="l0" />
-    <xacro:r_link prefix="l1" parent="l0" length="1.000000" radius="0.100000" joint_rpy="0 0 0" joint_xyz="0 0 0" link_rpy="0 0 0" link_xyz="0 0 0.500000"/>
-    <xacro:f_link prefix="l2" parent="l1" length="0.200000" radius="0.100000" link_rpy="0 1.570796 0" link_xyz="0.100000 0 1.000000"/>
-    <xacro:r_link prefix="l3" parent="l2" length="0.2" radius="0.100000" joint_rpy="1.570796 0 0" joint_xyz="0.200000 0 1.000000" link_rpy="0 0 0" link_xyz="0 0 0.000000"/>
-    <xacro:f_link prefix="l4" parent="l3" length="1.000000" radius="0.100000" link_rpy="0 1.570796 0" link_xyz="0.500000 0 0.000000"/>
-    <xacro:r_link prefix="l5" parent="l4" length="0.2" radius="0.100000" joint_rpy="0.000000 0 0" joint_xyz="1.000000 0 0.000000" link_rpy="0 0 0" link_xyz="0 0 0.000000"/>
-    <xacro:f_link prefix="l6" parent="l5" length="0.200000" radius="0.100000" link_rpy="0 1.570796 0" link_xyz="0.100000 0 0.000000"/>
-    <xacro:p_link prefix="l7" parent="l6" length="1.500000" radius="0.080000" joint_rpy="1.570796 0 0" joint_xyz="0.200000 0 0.000000" link_rpy="0 0 0" link_xyz="0 0 -0.750000"/>
+    <xacro:r_link prefix="l1" parent="l0" length="1.280000" radius="0.200000" joint_rpy="0 0 0" joint_xyz="0 0 0" link_rpy="0 0 0" link_xyz="0 0 0.640000"/>
+    <xacro:r_link prefix="l2" parent="l1" length="0.2" radius="0.200000" joint_rpy="-1.570796 0 0" joint_xyz="0.000000 0 1.280000" link_rpy="0 0 0" link_xyz="0 0 0.000000"/>
+    <xacro:f_link prefix="l3" parent="l2" length="-6.127000" radius="0.200000" joint_xyz="0 0 0" link_rpy="0 1.570796 0" link_xyz="-3.063500 0 0.000000"/>
+    <xacro:r_link prefix="l4" parent="l3" length="0.2" radius="0.200000" joint_rpy="0.000000 0 0" joint_xyz="-6.127000 0 0.000000" link_rpy="0 0 0" link_xyz="0 0 0.000000"/>
+    <xacro:f_link prefix="l5" parent="l4" length="5.716000" radius="0.200000" joint_xyz="0 0 0" link_rpy="0 1.570796 0" link_xyz="2.858000 0 0.000000"/>
+    <xacro:r_link prefix="l6" parent="l5" length="1.639000" radius="0.200000" joint_rpy="3.141593 0 0" joint_xyz="5.716000 0 0.000000" link_rpy="0 0 0" link_xyz="0 0 0.819500"/>
+    <xacro:r_link prefix="l7" parent="l6" length="-1.157000" radius="0.200000" joint_rpy="1.570796 0 0" joint_xyz="0.000000 0 1.639000" link_rpy="0 0 0" link_xyz="0 0 -0.578500"/>
+    <xacro:r_link prefix="l8" parent="l7" length="0.922000" radius="0.200000" joint_rpy="-1.570796 0 0" joint_xyz="0.000000 0 -1.157000" link_rpy="0 0 0" link_xyz="0 0 0.461000"/>
+    <xacro:f_link prefix="l9" parent="l8" length="0.000000" radius="0.200000" joint_xyz="0.000000 0 0.922000" link_rpy="0 1.570796 0" link_xyz="-0.000000 0 0"/>
+    <xacro:claw parent="l9" xyz="1.284000 0 0" scale="0.030000 0.030000 0.030000"/>
     <gazebo>
         <plugin name="gazebo_ros_control" filename="libgazebo_ros_control.so">
