Commit message: fixed end effector position problem. changed joints effort to resist gravity better

File: urdf/claw.xacro (robot description, xacro)
@@ -1,8 +1,8 @@
 <?xml version="1.0"?>
 <robot xmlns:xacro="http://www.ros.org/wiki/xacro" name="my_robot">
-<xacro:macro name="claw" params="parent xyz scale">
+<xacro:macro name="claw" params="parent rpy xyz scale">
 	<link name="claw">
         <visual>
-            <origin rpy="0 0 0" xyz="${xyz}"/>
+            <origin rpy="${rpy}" xyz="${xyz}"/>
             <geometry>
                 <mesh filename="package://project_rp/urdf/Claw.stl" scale="${scale}"/>

File: urdf/main.xacro (robot description, xacro)
@@ -7,14 +7,13 @@
     <xacro:include filename="$(find project_rp)/urdf/claw.xacro" />
     <xacro:base name="l0" />
-    <xacro:r_link prefix="l1" parent="l0" length="1.280000" radius="0.200000" joint_rpy="0 0 0" joint_xyz="0 0 0" link_rpy="0 0 0" link_xyz="0 0 0.640000"/>
-    <xacro:r_link prefix="l2" parent="l1" length="0.2" radius="0.200000" joint_rpy="-1.570796 0 0" joint_xyz="0.000000 0 1.280000" link_rpy="0 0 0" link_xyz="0 0 0.000000"/>
-    <xacro:f_link prefix="l3" parent="l2" length="-6.127000" radius="0.200000" joint_xyz="0 0 0" link_rpy="0 1.570796 0" link_xyz="-3.063500 0 0.000000"/>
-    <xacro:r_link prefix="l4" parent="l3" length="0.2" radius="0.200000" joint_rpy="0.000000 0 0" joint_xyz="-6.127000 0 0.000000" link_rpy="0 0 0" link_xyz="0 0 0.000000"/>
-    <xacro:f_link prefix="l5" parent="l4" length="5.716000" radius="0.200000" joint_xyz="0 0 0" link_rpy="0 1.570796 0" link_xyz="2.858000 0 0.000000"/>
-    <xacro:r_link prefix="l6" parent="l5" length="1.639000" radius="0.200000" joint_rpy="3.141593 0 0" joint_xyz="5.716000 0 0.000000" link_rpy="0 0 0" link_xyz="0 0 0.819500"/>
-    <xacro:r_link prefix="l7" parent="l6" length="-1.157000" radius="0.200000" joint_rpy="1.570796 0 0" joint_xyz="0.000000 0 1.639000" link_rpy="0 0 0" link_xyz="0 0 -0.578500"/>
-    <xacro:r_link prefix="l8" parent="l7" length="0.922000" radius="0.200000" joint_rpy="-1.570796 0 0" joint_xyz="0.000000 0 -1.157000" link_rpy="0 0 0" link_xyz="0 0 0.461000"/>
-    <xacro:f_link prefix="l9" parent="l8" length="0.000000" radius="0.200000" joint_xyz="0.000000 0 0.922000" link_rpy="0 1.570796 0" link_xyz="-0.000000 0 0"/>
-    <xacro:claw parent="l9" xyz="1.284000 0 0" scale="0.030000 0.030000 0.030000"/>
+    <xacro:p_link prefix="l1" parent="l0" length="2.000000" radius="0.080000" joint_rpy="0 0 0" joint_xyz="0 0 0" link_rpy="0 0 0" link_xyz="0 0 -1.000000"/>
+    <xacro:f_link prefix="l2" parent="l1" length="1.000000" radius="0.100000" joint_xyz="0 0 0" link_rpy="0 1.570796 0" link_xyz="0.500000 0 0.000000"/>
+    <xacro:r_link prefix="l3" parent="l2" length="0.2" radius="0.100000" joint_rpy="-1.570796 0 0" joint_xyz="1.000000 0 0.000000" link_rpy="0 0 0" link_xyz="0 0 0.000000"/>
+    <xacro:f_link prefix="l4" parent="l3" length="1.000000" radius="0.100000" joint_xyz="0 0 0" link_rpy="0 1.570796 0" link_xyz="0.500000 0 0.000000"/>
+    <xacro:r_link prefix="l5" parent="l4" length="0.2" radius="0.100000" joint_rpy="0.000000 0 0" joint_xyz="1.000000 0 0.000000" link_rpy="0 0 0" link_xyz="0 0 0.000000"/>
+    <xacro:f_link prefix="l6" parent="l5" length="1.000000" radius="0.100000" joint_xyz="0 0 0" link_rpy="0 1.570796 0" link_xyz="0.500000 0 0.000000"/>
+    <xacro:r_link prefix="l7" parent="l6" length="0.2" radius="0.100000" joint_rpy="0.000000 0 0" joint_xyz="1.000000 0 0.000000" link_rpy="0 0 0" link_xyz="0 0 0.000000"/>
+    <xacro:f_link prefix="l8" parent="l7" length="1.000000" radius="0.100000" joint_xyz="0 0 0" link_rpy="0 1.570796 0" link_xyz="0.500000 0 0.000000"/>
+    <xacro:claw parent="l8" rpy="0 1.570796 0" xyz="1.000000 0 -0.642000" scale="0.015000 0.015000 0.015000"/>
     <gazebo>
         <plugin name="gazebo_ros_control" filename="libgazebo_ros_control.so">

File: urdf/p_link.xacro (robot description, xacro)
@@ -20,5 +20,5 @@
         <child link="${prefix}"/>
         <origin rpy="${joint_rpy}" xyz="${joint_xyz}"/> <!-- move the child_frame with respect to parent_frame -->
-        <limit upper="${length}" effort="30" velocity="1.0"/>
+        <limit upper="${length}" effort="300" velocity="1.0"/>
         <dynamics damping="0.5" friction="0.0"/>
     </joint>

File: urdf/r_link.xacro (robot description, xacro)
@@ -20,5 +20,5 @@
         <child link="${prefix}"/>
         <origin rpy="${joint_rpy}" xyz="${joint_xyz}"/>
-        <limit effort="30" velocity="1.0"/>
+        <limit effort="300" velocity="1.0"/>
         <dynamics damping="0.5" friction="0.0"/>
     </joint>
